File: pcb/gb_video_breakout/gb_video_breakout.kicad_pcb (KiCad board)
At the start: 11 copper layers, 19.6 x 22.4 mm, 12 parts, among them J1 Conn_01x05, Q1 MMBF170, Q2 MMBF170, U1 SN74LVC1G17QDCKRQ1, U2 SN74LVC1G17QDCKRQ1

Commit message: V0.5
Parts:
- removed LED_3V3: HSMS-C177, LED_SMD:LED_1206_3216Metric
- removed LED_5V1: HSMG-C177, LED_SMD:LED_1206_3216Metric
- removed Q1, Q2: MMBF170, Package_TO_SOT_SMD:SOT-23
- removed R1, R5: RES 1K OHM 1%, Resistor_SMD:R_1206_3216Metric
- added C1: C, Capacitor_SMD:C_0805_2012Metric, F.Cu at (147.8, 84.9)
- added C2: C, Capacitor_SMD:C_0805_2012Metric, F.Cu at (141.7, 84.7)
- added D1: LED, LED_SMD:LED_0805_2012Metric, F.Cu at (150.5, 88.8)
- added D2: LED, LED_SMD:LED_0805_2012Metric, F.Cu at (138.9, 85.4)
- added U3: SN74LVC1G17QDCKRQ1, SN74LVC:SOT65P210X110-5N, F.Cu at (147.2, 87.8)
- R3: value RES 360 OHM 1/8W 5% -> R; footprint Resistor_SMD:R_1206_3216Metric -> Resistor_SMD:R_0805_2012Metric
- R4: value RES 240 OHM 1/8W 5% -> R; footprint Resistor_SMD:R_1206_3216Metric -> Resistor_SMD:R_0805_2012Metric
- U1, U2: footprint SN74LVC1G17:SOT65P210X110-5N -> SN74LVC:SOT65P210X110-5N
- moved R3 13.7 mm to (150.5, 85.5)
- moved R4 11.6 mm to (138.9, 88.8)
- moved J1 6.14 mm to (139.4, 81.8)
- moved U2 5.22 mm to (144.5, 87.8)
- moved U1 5.09 mm to (141.8, 87.8)
Connections:
- net SI_3V3 renamed RX_3V3
- net SI_5V renamed RX_5V
- net SO_3V3 renamed TX_3V3
- net SO_5V renamed TX_5V
- GB1 pad 1: +5V -> unconnected-(GB1-VDD35-Pad1)
- GB1 pad 4: unconnected-(GB1-SD-Pad4) -> +5V
- GB1 pad 5: SC_5V -> CLK_5V
- J1 pad 4: SC_3V3 -> CLK_3V3
Routing:
- net GND: track 16.8 -> 2.40 mm, vias 5 -> 17
- net SC_5V: track 9.32 -> 0.00 mm, vias 1 -> 0
- net SC_3V3: track 6.53 -> 0.00 mm
- net RX_5V: track 11.0 -> 5.25 mm
- net CLK_5V: track 0.00 -> 5.52 mm, vias 0 -> 1
- net CLK_3V3: track 0.00 -> 5.31 mm
- net TX_5V: track 10.4 -> 6.30 mm
- net Net-(Q1-D): track 3.25 -> 0.00 mm
- net Net-(D2-K): track 3.87 -> 1.51 mm
- net +5V: track 22.7 -> 20.4 mm, vias 4 -> 0
- net Net-(D1-K): track 3.84 -> 1.53 mm
- net TX_3V3: track 6.16 -> 5.14 mm
- net +3V3: track 16.9 -> 17.7 mm, vias 2 -> 3
- added copper zone on F.Cu, net GND
- removed copper zone on F.Cu, net +3V3
- removed copper zone on F.Cu, net +5V
Other:
- board size 19.6 x 22.4 mm -> 14.6 x 17.3 mm
- board text added: "3V3"
- board text added: "CLK"
- board text added: "GND"
- board text added: "RX"
- board text added: "TX"
- board text added: "v0.5"
- board text removed: "2024"
- board text removed: "ChromaLock"
- board text removed: "GBLINK v0.1"

Commit message: restructure
Routing:
- net Net-(D1-K): track 1.53 -> 2.12 mm
Changed lines of the file:
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@@
 		(tags "capacitor")
 		(property "Reference" "C1"
-			(at -0.05 -0.05 360)
+			(at -0.05 -0.05 0)
 			(layer "F.SilkS")
 			(hide yes)
@@
 		)
 		(property "Value" "C"
-			(at 0 1.68 360)
+			(at 0 1.68 0)
 			(layer "F.Fab")
 			(effects
@@
 		)
 		(fp_text user "${REFERENCE}"
-			(at 0 0 360)
+			(at 0 0 0)
 			(layer "F.Fab")
 			(effects
@@
 	)
 	(segment
-		(start 149.925 87.8375)
-		(end 149.925 86.3125)
+		(start 150.5 86.8875)
+		(end 150.5 86.3625)
+		(width 0.25)
+		(layer "F.Cu")
+		(net 1)
+	)
+	(segment
+		(start 150.5 87.8875)
+		(end 150.5 86.3625)
+		(width 0.25)
+		(layer "F.Cu")
+		(net 1)
+	)
+	(segment
+		(start 150.5 86.3625)
+		(end 150.55 86.4125)
 		(width 0.25)
 		(layer "F.Cu")
@@
 	)
 	(via
-		(at 148.6 86.75)
+		(at 148.6 87)
 		(size 0.8)
 		(drill 0.4)
@@
 	)
 	(via
-		(at 140.7 90.35)
+		(at 140.5 90.15)
 		(size 0.8)
 		(drill 0.4)
@@
 	)
 	(segment
-		(start 144.5 94)
-		(end 144.5 91.9)
+		(start 149.35 86.4)
+		(end 149.35 87.55)
 		(width 0.25)
 		(layer "F.Cu")
@@
 	(segment
 		(start 148.8 84.9)
-		(end 149.35 85.45)
-		(width 0.25)
-		(layer "F.Cu")
-		(net 3)
-	)
-	(segment
-		(start 144.5 91.9)
-		(end 144.5 91.05)
-		(width 0.25)
-		(layer "F.Cu")
-		(net 3)
-	)
-	(segment
-		(start 144.2 91.05)
-		(end 142.5 89.35)
+		(end 148.8 85.85)
 		(width 0.25)
 		(layer "F.Cu")
@@
 	)
 	(segment
-		(start 144.5 91.05)
-		(end 144.2 91.05)
+		(start 144.5 94)
+		(end 144.5 91.35)
 		(width 0.25)
 		(layer "F.Cu")
@@
 	)
 	(segment
+		(start 148.8 85.85)
+		(end 149.35 86.4)
+		(width 0.25)
+		(layer "F.Cu")
+		(net 3)
+	)
+	(segment
 		(start 149.126 87.776)
 		(end 149.35 88)
@@
 	)
 	(segment
-		(start 149.35 85.45)
-		(end 149.35 87.55)
-		(width 0.25)
-		(layer "F.Cu")
-		(net 3)
-	)
-	(segment
 		(start 149.1 87.776)
 		(end 149.126 87.776)
@@
 	)
 	(segment
+		(start 142.5 89.35)
+		(end 142.5 88.75)
+		(width 0.25)
+		(layer "F.Cu")
+		(net 3)
+	)
+	(segment
+		(start 144.5 91.35)
+		(end 142.5 89.35)
+		(width 0.25)
+		(layer "F.Cu")
+		(net 3)
+	)
+	(segment
 		(start 149.35 88)
 		(end 149.35 88.967823)
-		(width 0.25)
-		(layer "F.Cu")
-		(net 3)
-	)
-	(segment
-		(start 142.5 89.35)
-		(end 142.5 88.75)
 		(width 0.25)
 		(layer "F.Cu")
@@
 		(polygon
 			(pts
-				(xy 134.15 77.6) (xy 156.7 78.85) (xy 155.4 98.1) (xy 135.85 98.5)
+				(xy 137 79) (xy 152 79) (xy 152 92) (xy 137 92)
 			)
 		)
@@
 		(polygon
 			(pts
-				(xy 133.55 76.8) (xy 157.5 77.75) (xy 152.8 100.1) (xy 134.25 100.25)
-			)
-		)
+				(xy 137 79) (xy 152 79) (xy 152 92) (xy 137 92)
+			)
+		)

Commit message: rearrange
Routing:
- net GND: track 2.40 -> 5.31 mm
Changed lines of the file:
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@@
+		(net 2)
+	)
+	(segment
+		(start 146.5 92.9)
+		(end 145.5 91.9)
+		(width 0.25)
+		(layer "F.Cu")
+		(net 2)
+	)
+	(segment
+		(start 145.5 91.9)
+		(end 145.5 91.5)
+		(width 0.25)
+		(layer "F.Cu")
+		(net 2)
+	)
+	(segment
+		(start 146.5 94)
+		(end 146.5 92.9)
+		(width 0.25)
+		(layer "F.Cu")
 		(net 2)
 	)
@@
 		(polygon
 			(pts
-				(xy 137 79) (xy 152 79) (xy 152 92) (xy 137 92)
+				(xy 137 79.5) (xy 152 79.5) (xy 152 92) (xy 137 92)
 			)
 		)
@@
 		(polygon
 			(pts
-				(xy 137 79) (xy 152 79) (xy 152 92) (xy 137 92)
+				(xy 137 79.5) (xy 152 79.5) (xy 152 92) (xy 137 92)
 			)
 		)
