File: pcb/gb_video_pico_breakout/gb_video_pico_breakout.kicad_sch (KiCad schematic)
At the start: 19 parts, among them J1 Conn_01x05, U1 SN74LVC1G17QDCKRQ1, U2 SN74LVC1G17QDCKRQ1, U3 SN74LVC1G17QDCKRQ1, U4 Pico

Commit message: add serialtransfer support
Parts:
- removed D1: LED, LED_SMD:LED_0805_2012Metric, symbol LEDC2012X50N:HSMG-C177
- added D1: LED, LED_SMD:LED_0805_2012Metric, symbol Device:LED
- D2: symbol LEDC2012X50N:HSMG-C177 -> Device:LED
Connections:
- net +5V: now also D1.2 (A)
- net at R3.1: now also D1.1 (K)
Other:
- moved on the sheet: C1, C2, R3, R4, TP1, TP2, TP3
