File: pcb/gb_video_pico_breakout/gb_video_pico_breakout.kicad_pcb (KiCad board)
At the start: 11 copper layers, 44 x 73 mm, 19 parts, among them J1 Conn_01x05, U1 SN74LVC1G17QDCKRQ1, U2 SN74LVC1G17QDCKRQ1, U3 SN74LVC1G17QDCKRQ1, U4 Pico

Commit message: add color
Parts:
- removed JP1, JP2, JP3, JP4: SolderJumper_2_Open, Jumper:SolderJumper-2_P1.3mm_Open_RoundedPad1.0x1.5mm
Connections:
- J1 pad 1: Net-(J1-Pin_1) -> +3V3
- J1 pad 2: Net-(J1-Pin_2) -> TX_3V3
- J1 pad 3: Net-(J1-Pin_3) -> RX_3V3
- J1 pad 4: Net-(J1-Pin_4) -> CLK_3V3
- U4 pad 36: Net-(J1-Pin_1) -> +3V3
- U4 pad 4: Net-(J1-Pin_3) -> RX_3V3
- U4 pad 5: Net-(J1-Pin_4) -> CLK_3V3
- U4 pad 6: Net-(J1-Pin_2) -> TX_3V3
Routing:
- net RX_3V3: track 3.18 -> 57.9 mm, vias 0 -> 2
- net Net-(J1-Pin_1): track 54.1 -> 0.00 mm
- net CLK_3V3: track 3.63 -> 57.7 mm, vias 0 -> 2
- net Net-(J1-Pin_3): track 53.4 -> 0.00 mm, vias 2 -> 0
- net Net-(J1-Pin_4): track 52.8 -> 0.00 mm, vias 2 -> 0
- net +3V3: track 27.6 -> 79.8 mm
- net TX_3V3: track 3.35 -> 52.9 mm, vias 0 -> 2
- net Net-(J1-Pin_2): track 48.3 -> 0.00 mm, vias 2 -> 0
Other:
- board text added: "GB"
- board text added: "Pico"
